Commit message: Scara.urdf from medium

File: urdf/scara.urdf (robot description, URDF)
Before this commit: robot myfirst, 1 links, 0 joints
Links:
- added link arm1; visual box size=0.1 1.0 0.1
- added link arm2; visual box size=0.1 0.5 0.1
- added link world
- link base_link: geometry visual cylinder length=0.8 radius=0.1
Joints:
- added joint arm1_joint: type revolute, parent base_link, child arm1, origin xyz=0.0 0.0 0.8 rpy=0.0 0.0 0.0, axis 0.0 0.0 1.0, limit lower=-1.0 upper=1.0 effort=1000.0 velocity=1000.0
- added joint arm2_joint: type revolute, parent arm1, child arm2, origin xyz=0.0 -1.0 0.0 rpy=0.0 0.0 0.0, axis 0.0 0.0 1.0, limit lower=-1.0 upper=1.0 effort=1000.0 velocity=1000.0
- added joint base_joint: type fixed, parent world, child base_link

Commit message: Build Scara Robot without Endeffector

File: urdf/scara.urdf (robot description, URDF)
Before this commit: robot scara_robot, 4 links, 3 joints
Links:
- removed link arm1
- removed link arm2
- added link arm1_connection; visual cylinder length=0.5 radius=0.05
- added link arm1_cylinder; visual cylinder length=0.2 radius=0.1
- added link arm2_connection; visual cylinder length=0.5 radius=0.05
- added link arm2_cylinder1; visual cylinder length=0.2 radius=0.1
- added link arm2_cylinder2; visual cylinder length=0.2 radius=0.1
- added link arm3_cylinder1; visual cylinder length=0.2 radius=0.1
- added link arm3_prismatic; visual cylinder length=0.5 radius=0.075
Joints:
- removed joint arm1_joint
- added joint arm1_joint_Gelenk: type revolute, parent base_link, child arm1_cylinder, origin xyz=0.0 0.0 0.8 rpy=0.0 0.0 0.0, axis 0.0 0.0 1.0, limit lower=-1.0 upper=1.0 effort=1000.0 velocity=1000.0
- added joint arm1_joint_box: type fixed, parent arm1_cylinder, child arm1_connection
- added joint arm2_joint_Gelenk: type fixed, parent arm1_connection, child arm2_cylinder1, origin xyz=0.5 0.0 0.0 rpy=0.0 0.0 0.0
- added joint arm2_joint_box: type fixed, parent arm2_cylinder2, child arm2_connection
- added joint arm3_joint: type prismatic, parent arm3_cylinder1, child arm3_prismatic, origin xyz=0.0 0.0 0.1 rpy=0.0 0.0 0.0, axis 0.0 0.0 1.0, limit lower=-0.150 upper=0.150 effort=1000.0 velocity=1000.0
- added joint arm3_joint_Gelenk: type fixed, parent arm2_connection, child arm3_cylinder1, origin xyz=0.5 0.0 0.0 rpy=0.0 0.0 0.0
- joint arm2_joint: child arm2 -> arm2_cylinder2; origin xyz=0.0 -1.0 0.0 rpy=0.0 0.0 0.0 -> xyz=0.0 0.0 0.2 rpy=0.0 0.0 0.0; parent arm1 -> arm2_cylinder1

Commit message: Scara Robot complete

File: urdf/scara.urdf (robot description, URDF)
Before this commit: robot scara_robot, 9 links, 8 joints
Links:
- added link Hand_Base; visual box size=0.1 0.1 0.1
- added link arm3_connection; visual cylinder length=0.1 radius=0.025
Joints:
- added joint Hand_Base_joint: type fixed, parent arm3_connection, child Hand_Base, origin xyz=0.0 0.0 -0.15 rpy=0.0 0.0 0.0
- added joint arm3_joint_box: type revolute, parent arm3_prismatic, child arm3_connection, origin xyz=0.0 0.0 -0.55 rpy=0.0 0.0 0.0, axis 0.0 0.0 1.0, limit lower=-1.5 upper=1.5 effort=1000.0 velocity=1000.0
- joint arm1_joint_Gelenk: origin xyz=0.0 0.0 0.8 rpy=0.0 0.0 0.0 -> xyz=0.0 0.0 0.9 rpy=0.0 0.0 0.0
- joint arm1_joint_box: origin (none) -> xyz=0.25 0.0 0.0 rpy=0.0 0.0 0.0
- joint arm2_joint_Gelenk: origin xyz=0.5 0.0 0.0 rpy=0.0 0.0 0.0 -> xyz=0.25 0.0 0.0 rpy=0.0 0.0 0.0
- joint arm2_joint_box: origin (none) -> xyz=0.25 0.0 0.0 rpy=0.0 0.0 0.0
- joint arm3_joint: limit lower=-0.150 upper=0.150 effort=1000.0 velocity=1000.0 -> lower=0.0 upper=0.3 effort=1000.0 velocity=1000.0
- joint arm3_joint_Gelenk: origin xyz=0.5 0.0 0.0 rpy=0.0 0.0 0.0 -> xyz=0.25 0.0 0.0 rpy=0.0 0.0 0.0

Commit message: final scara with xacro params

File: urdf/scara.urdf (robot description, URDF)
Before this commit: robot scara_robot, 11 links, 10 joints
Links:
- link arm1_connection: geometry visual cylinder length=0.6 radius=0.05
- link arm2_connection: geometry visual cylinder length=0.8 radius=0.05
- link arm3_prismatic: geometry visual cylinder length=0.4999999999999998 radius=0.075
- link base_link: geometry visual cylinder length=1 radius=0.1
Joints:
- joint Hand_Base_joint: origin xyz=0.0 0.0 -0.15 rpy=0.0 0.0 0.0 -> xyz=0.0 0.0 -0.15000000000000002 rpy=0.0 0.0 0.0
- joint arm1_joint_Gelenk: axis 0.0 0.0 1.0 -> 0.0 0.0 1.2; origin xyz=0.0 0.0 0.9 rpy=0.0 0.0 0.0 -> xyz=0.0 0.0 1.1 rpy=0.0 0.0 0.0
- joint arm1_joint_box: origin xyz=0.25 0.0 0.0 rpy=0.0 0.0 0.0 -> xyz=0.3 0.0 0.0 rpy=0.0 0.0 0.0
- joint arm2_joint_Gelenk: origin xyz=0.25 0.0 0.0 rpy=0.0 0.0 0.0 -> xyz=0.3 0.0 0.0 rpy=0.0 0.0 0.0
- joint arm2_joint_box: origin xyz=0.25 0.0 0.0 rpy=0.0 0.0 0.0 -> xyz=0.4 0.0 0.0 rpy=0.0 0.0 0.0
- joint arm3_joint: limit lower=0.0 upper=0.3 effort=1000.0 velocity=1000.0 -> lower=0.0 upper=0.29999999999999977 effort=1000.0 velocity=1000.0
- joint arm3_joint_Gelenk: origin xyz=0.25 0.0 0.0 rpy=0.0 0.0 0.0 -> xyz=0.4 0.0 0.0 rpy=0.0 0.0 0.0
- joint arm3_joint_box: origin xyz=0.0 0.0 -0.55 rpy=0.0 0.0 0.0 -> xyz=0.0 0.0 -0.5499999999999998 rpy=0.0 0.0 0.0

Commit message: Task 5.3 and 5.4

File: urdf/scara.urdf (robot description, URDF)
Before this commit: robot scara_robot, 11 links, 10 joints
Joints:
- joint arm3_joint_box: mimic (none) -> joint=arm1_joint_Gelenk multiplier=1 offset=1

File: urdf/scara.urdf.xacro (robot description, xacro)
@@ -154,4 +154,5 @@
             <child link="arm3_connection"/>
             <axis xyz="0.0 0.0 1.0"/>
+            <mimic joint="arm1_joint_Gelenk" multiplier="1" offset="1"/>
             <limit lower="-1.5" upper="1.5" effort="1000.0" velocity="1000.0"/>
     </joint>
